File: LoRa.kicad_sch (KiCad schematic)
At the start: 0 parts

Commit message: Footprint
Parts:
- added U3: RAK3172, symbol RAK3172:RAK3172
Changed lines of the file:
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@@
 	(generator_version "8.0")
 	(paper "A4")
+	(symbol
+		(lib_id "RAK3172:RAK3172")
+		(at 132.08 64.77 0)
+		(unit 1)
+		(exclude_from_sim no)
+		(in_bom yes)
+		(on_board yes)
+		(dnp no)
+		(fields_autoplaced yes)
+		(property "Reference" "U3"
+			(at 149.5141 59.69 0)
+			(effects
+				(font
+					(size 1.27 1.27)
+				)
+				(justify left)
+			)
+		)
+		(property "Value" "RAK3172"
+			(at 149.5141 62.23 0)
+			(effects
+				(font
+					(size 1.27 1.27)
+				)
+				(justify left)
+			)
+		)
+		(property "Footprint" ""
+			(at 132.08 64.77 0)
+			(effects
+				(font
+					(size 1.27 1.27)
+				)
+				(hide yes)
+			)
+		)
+		(property "Datasheet" ""
+			(at 132.08 64.77 0)
+			(effects
+				(font
+					(size 1.27 1.27)
+				)
+				(hide yes)
+			)
+		)
+		(property "Description" ""
+			(at 132.08 64.77 0)
+			(effects
+				(font
+					(size 1.27 1.27)
+				)
+				(hide yes)
+			)
+		)
+		(pin "9"
+		)
+		(pin "31"
+		)
+		(pin "16"
+		)
+		(pin "15"
+		)
+		(pin "14"
+		)
+		(pin "13"
+		)
+		(pin "12"
+		)
+		(pin "11"
+		)
+		(pin "10"
+		)
+		(pin "32"
+		)
+		(pin "1"
+		)
+		(pin "19"
+		)
+		(pin "24"
+		)
+		(pin "28"
+		)
+		(pin "20"
+		)
+		(pin "17"
+		)
+		(pin "29"
+		)
+		(pin "6"
+		)
+		(pin "18"
+		)
+		(pin "2"
+		)
+		(pin "5"
+		)
+		(pin "4"
+		)
+		(pin "22"
+		)
+		(pin "21"
+		)
+		(pin "7"
+		)
+		(pin "27"
+		)
+		(pin "25"
+		)
+		(pin "3"
+		)
+		(pin "26"
+		)
+		(pin "30"
+		)
+		(pin "23"
+		)
+		(pin "8"
+		)
+		(instances
+			(project ""
+				(path "/e0ffc31c-24f5-4303-8af9-d0625c9ddd62/2f968173-500b-405d-91c1-1d157a663cec"
+					(reference "U3")
+					(unit 1)
+				)
+			)
+		)
+	)
 )

Commit message: LoRa Scheme
Parts:
- added C11, C13: 100nF, symbol Device:C_Small
- added C14: 10uF, symbol Device:C_Small
- added D2: LED_Small, symbol Device:LED_Small
- added R2, R3: 10K, symbol Device:R_Small
- added R4: 4K7, symbol Device:R_Small
- added SW1, SW2: SW_Push, symbol Switch:SW_Push
Connections:
- net RAK_UART2_RX: now reaches U3.1 (UART2_RX)
- net GND: now reaches U3.11 (GND)
- net GND: now also U3.17 (GND), U3.18 (GND), U3.23 (GND), U3.28 (GND), C11.2, C13.2, C14.2, D2.1 (K), R3.2, SW1.1
- net RAK_UART2_TX: now reaches U3.2 (UART2_TX)
- net RAK_BOOT: now reaches U3.21 (BOOT)
- net RAK_BOOT: now also R3.1, SW2.2
- net RAK_RESET: now reaches U3.22 (RST)
- net RAK_RESET: now also C11.1, R2.2, SW1.2
- net LORA_3V3: now reaches U3.24 (VCC)
- net LORA_3V3: now also C13.1, C14.1, R2.1, R4.1, SW2.1
- net RAK_PB12: now reaches U3.27 (PB12)
- net RAK_PA0: now reaches U3.29 (PA0)
- net RAK_PB5: now reaches U3.30 (PB5)
- net RAK_UART1_TX: now reaches U3.4 (UART1_TX)
- net RAK_UART1_RX: now reaches U3.5 (UART1_RX)
- net RAK_PA1: now reaches U3.6 (PA1)
- new net: D2.2 (A), R4.2
- no-connect marks 0 -> 16
