File: Sensors.kicad_sch (KiCad schematic)
At the start: 0 parts

Commit message: sensor
Parts:
- added C12: 100nF, symbol Device:C_Small
- added R5, R6: 4K7, symbol Device:R_Small
- added U4: HDC1080, Package_SON:Texas_PWSON-N6, symbol Sensor_Humidity:HDC1080
Connections:
- new net GND: C12.2, U4.2 (GND)
- new net SENS_3V3: C12.1, R5.2, R6.1, U4.5 (VCC)
- new net SENS_SCL: R6.2, U4.6 (SCL)
- new net SENS_SDA: R5.1, U4.1 (SDA)
