File: LoRaNode328.kicad_sch (KiCad schematic)
At the start: 4 parts, among them U1 TPS62056DGS

Commit message: MCU
Parts:
- removed C2: C_Small, symbol Device:C_Small
- removed D2: SS24, Diode_SMD:D_SMA, symbol Diode:SS24
- removed L1: L_Small, symbol Device:L_Small
- removed U1: TPS62056DGS, Package_SO:VSSOP-10_3x3mm_P0.5mm, symbol Regulator_Switching:TPS62056DGS
Other:
- added sheet Connectors (Connectors.kicad_sch)
- added sheet LoRa (LoRa.kicad_sch)
- added sheet MCU (MCU.kicad_sch)
- added sheet Power_Control (Power_Control.kicad_sch)
- added sheet Power_Regulator (Power_Regulator.sch.kicad_sch)
- added sheet Sensors (Sensors.kicad_sch)

Commit message: Footprint
Changed lines of the file:
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@@
 	(paper "A4")
 	(sheet
-		(at 165.1 67.31)
+		(at 91.44 31.75)
 		(size 12.7 5.08)
 		(fields_autoplaced yes)
@@
 		)
 		(property "Sheetname" "LoRa"
-			(at 165.1 66.5984 0)
+			(at 91.44 31.0384 0)
 			(effects
 				(font
@@
 		)
 		(property "Sheetfile" "LoRa.kicad_sch"
-			(at 165.1 72.9746 0)
+			(at 91.44 37.4146 0)
 			(effects
 				(font

Commit message: LoRa Scheme
Other:
- sheet LoRa ports: added LORA_3V3, RAK_BOOT, RAK_PA0, RAK_PA1, RAK_PB12, RAK_PB5, RAK_RESET, RAK_UART1_RX, RAK_UART1_TX, RAK_UART2_RX, RAK_UART2_TX; removed none
- sheet MCU ports: added MCU_3V3; removed none
Changed lines of the file:
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@@
 	(paper "A4")
 	(sheet
-		(at 91.44 31.75)
-		(size 12.7 5.08)
+		(at 87.63 30.48)
+		(size 31.75 27.94)
 		(fields_autoplaced yes)
 		(stroke
@@
 		)
 		(property "Sheetname" "LoRa"
-			(at 91.44 31.0384 0)
+			(at 87.63 29.7684 0)
 			(effects
 				(font
@@
 		)
 		(property "Sheetfile" "LoRa.kicad_sch"
-			(at 91.44 37.4146 0)
+			(at 87.63 59.0046 0)
 			(effects
 				(font
@@
 				)
 				(justify left top)
+			)
+		)
+		(pin "LORA_3V3" input
+			(at 87.63 35.56 180)
+			(effects
+				(font
+					(size 1.27 1.27)
+				)
+				(justify left)
+			)
+		)
+		(pin "RAK_PB12" output
+			(at 119.38 43.18 0)
+			(effects
+				(font
+					(size 1.27 1.27)
+				)
+				(justify right)
+			)
+		)
+		(pin "RAK_PA1" output
+			(at 119.38 38.1 0)
+			(effects
+				(font
+					(size 1.27 1.27)
+				)
+				(justify right)
+			)
+		)
+		(pin "RAK_PB5" output
+			(at 119.38 40.64 0)
+			(effects
+				(font
+					(size 1.27 1.27)
+				)
+				(justify right)
+			)
+		)
+		(pin "RAK_PA0" output
+			(at 119.38 35.56 0)
+			(effects
+				(font
+					(size 1.27 1.27)
+				)
+				(justify right)
+			)
+		)
+		(pin "RAK_RESET" input
+			(at 87.63 39.37 180)
+			(effects
+				(font
+					(size 1.27 1.27)
+				)
+				(justify left)
+			)
+		)
+		(pin "RAK_UART1_RX" input
+			(at 87.63 45.72 180)
+			(effects
+				(font
+					(size 1.27 1.27)
+				)
+				(justify left)
+			)
+		)
+		(pin "RAK_UART1_TX" output
+			(at 87.63 48.26 180)
+			(effects
+				(font
+					(size 1.27 1.27)
+				)
+				(justify left)
+			)
+		)
+		(pin "RAK_BOOT" input
+			(at 87.63 41.91 180)
+			(effects
+				(font
+					(size 1.27 1.27)
+				)
+				(justify left)
+			)
+		)
+		(pin "RAK_UART2_TX" output
+			(at 87.63 54.61 180)
+			(effects
+				(font
+					(size 1.27 1.27)
+				)
+				(justify left)
+			)
+		)
+		(pin "RAK_UART2_RX" input
+			(at 87.63 52.07 180)
+			(effects
+				(font
+					(size 1.27 1.27)
+				)
+				(justify left)
 			)
 		)
@@
 	)
 	(sheet
-		(at 191.77 30.48)
+		(at 138.43 30.48)
 		(size 12.7 5.08)
 		(fields_autoplaced yes)
@@
 		)
 		(property "Sheetname" "Sensors"
-			(at 191.77 29.7684 0)
+			(at 138.43 29.7684 0)
 			(effects
 				(font
@@
 		)
 		(property "Sheetfile" "Sensors.kicad_sch"
-			(at 191.77 36.1446 0)
+			(at 138.43 36.1446 0)
 			(effects
 				(font
@@
 	)
 	(sheet
-		(at 191.77 60.96)
+		(at 138.43 60.96)
 		(size 12.7 5.08)
 		(fields_autoplaced yes)
@@
 		)
 		(property "Sheetname" "Connectors"
-			(at 191.77 60.2484 0)
+			(at 138.43 60.2484 0)
 			(effects
 				(font
@@
 		)
 		(property "Sheetfile" "Connectors.kicad_sch"
-			(at 191.77 66.6246 0)
+			(at 138.43 66.6246 0)
 			(effects
 				(font
@@
 			)
 		)
+		(pin "MCU_3V3" input
+			(at 35.56 58.42 180)
+			(effects
+				(font
+					(size 1.27 1.27)
+				)
+				(justify left)
+			)
+		)
 		(instances
 			(project "LoRaNode328"
@@
 	)
 	(sheet
-		(at 191.77 45.72)
+		(at 138.43 45.72)
 		(size 12.7 5.08)
 		(fields_autoplaced yes)
@@
 		)
 		(property "Sheetname" "Power_Control"
-			(at 191.77 45.0084 0)
+			(at 138.43 45.0084 0)
 			(effects
 				(font
@@
 		)
 		(property "Sheetfile" "Power_Control.kicad_sch"
-			(at 191.77 51.3846 0)
-			(effects
-				(font
+			(at 138.43 51.3846 0)
+			(effects
+				(font

Commit message: sensor
Other:
- sheet Sensors ports: added SENS_3V3, SENS_SCL, SENS_SDA; removed none
Changed lines of the file:
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@@
 	)
 	(sheet
-		(at 138.43 30.48)
+		(at 88.9 67.31)
+		(size 17.78 15.24)
+		(fields_autoplaced yes)
+		(stroke
+			(width 0.1524)
+			(type solid)
+		)
+		(fill
+			(color 0 0 0 0.0000)
+		)
+		(property "Sheetname" "Sensors"
+			(at 88.9 66.5984 0)
+			(effects
+				(font
+					(size 1.27 1.27)
+				)
+				(justify left bottom)
+			)
+		)
+		(property "Sheetfile" "Sensors.kicad_sch"
+			(at 88.9 83.1346 0)
+			(effects
+				(font
+					(size 1.27 1.27)
+				)
+				(justify left top)
+			)
+		)
+		(pin "SENS_3V3" input
+			(at 88.9 72.39 180)
+			(effects
+				(font
+					(size 1.27 1.27)
+				)
+				(justify left)
+			)
+		)
+		(pin "SENS_SCL" input
+			(at 88.9 74.93 180)
+			(effects
+				(font
+					(size 1.27 1.27)
+				)
+				(justify left)
+			)
+		)
+		(pin "SENS_SDA" input
+			(at 88.9 77.47 180)
+			(effects
+				(font
+					(size 1.27 1.27)
+				)
+				(justify left)
+			)
+		)
+		(instances
+			(project "LoRaNode328"
+				(path "/e0ffc31c-24f5-4303-8af9-d0625c9ddd62"
+					(page "5")
+				)
+			)
+		)
+	)
+	(sheet
+		(at 137.16 31.75)
 		(size 12.7 5.08)
 		(fields_autoplaced yes)
@@
 			(color 0 0 0 0.0000)
 		)
-		(property "Sheetname" "Sensors"
-			(at 138.43 29.7684 0)
+		(property "Sheetname" "Connectors"
+			(at 137.16 31.0384 0)
 			(effects
 				(font
@@
 			)
 		)
-		(property "Sheetfile" "Sensors.kicad_sch"
-			(at 138.43 36.1446 0)
-			(effects
-				(font
-					(size 1.27 1.27)
-				)
-				(justify left top)
-			)
-		)
-		(instances
-			(project "LoRaNode328"
-				(path "/e0ffc31c-24f5-4303-8af9-d0625c9ddd62"
-					(page "5")
-				)
-			)
-		)
-	)
-	(sheet
-		(at 138.43 60.96)
-		(size 12.7 5.08)
-		(fields_autoplaced yes)
-		(stroke
-			(width 0.1524)
-			(type solid)
-		)
-		(fill
-			(color 0 0 0 0.0000)
-		)
-		(property "Sheetname" "Connectors"
-			(at 138.43 60.2484 0)
-			(effects
-				(font
-					(size 1.27 1.27)
-				)
-				(justify left bottom)
-			)
-		)
 		(property "Sheetfile" "Connectors.kicad_sch"
-			(at 138.43 66.6246 0)
+			(at 137.16 37.4146 0)
 			(effects
 				(font
@@
 	)
 	(sheet
-		(at 138.43 45.72)
+		(at 119.38 68.58)
 		(size 12.7 5.08)
 		(fields_autoplaced yes)
@@
 		)
 		(property "Sheetname" "Power_Control"
-			(at 138.43 45.0084 0)
+			(at 119.38 67.8684 0)
 			(effects
 				(font
@@
 		)
 		(property "Sheetfile" "Power_Control.kicad_sch"
-			(at 138.43 51.3846 0)
-			(effects
-				(font
+			(at 119.38 74.2446 0)
+			(effects
+				(font

Commit message: load control
Other:
- sheet Power_Control ports: added LC_3V3, LOAD1_3V3, LOAD1_EN, LOAD2_3V3, LOAD2_EN, LORA_3V3, LORA_EN, SENS_3V3, SENS_EN; removed none
Changed lines of the file:
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@@
 	)
 	(sheet
-		(at 119.38 68.58)
-		(size 12.7 5.08)
+		(at 87.63 92.71)
+		(size 33.02 21.59)
 		(fields_autoplaced yes)
 		(stroke
@@
 		)
 		(property "Sheetname" "Power_Control"
-			(at 119.38 67.8684 0)
+			(at 87.63 91.9984 0)
 			(effects
 				(font
@@
 		)
 		(property "Sheetfile" "Power_Control.kicad_sch"
-			(at 119.38 74.2446 0)
+			(at 87.63 114.8846 0)
 			(effects
 				(font
@@
 			)
 		)
+		(pin "LC_3V3" input
+			(at 87.63 97.79 180)
+			(effects
+				(font
+					(size 1.27 1.27)
+				)
+				(justify left)
+			)
+		)
+		(pin "LORA_EN" input
+			(at 87.63 100.33 180)
+			(effects
+				(font
+					(size 1.27 1.27)
+				)
+				(justify left)
+			)
+		)
+		(pin "SENS_EN" input
+			(at 87.63 102.87 180)
+			(effects
+				(font
+					(size 1.27 1.27)
+				)
+				(justify left)
+			)
+		)
+		(pin "SENS_3V3" output
+			(at 120.65 102.87 0)
+			(effects
+				(font
+					(size 1.27 1.27)
+				)
+				(justify right)
+			)
+		)
+		(pin "LORA_3V3" output
+			(at 120.65 100.33 0)
+			(effects
+				(font
+					(size 1.27 1.27)
+				)
+				(justify right)
+			)
+		)
+		(pin "LOAD2_3V3" output
+			(at 120.65 107.95 0)
+			(effects
+				(font
+					(size 1.27 1.27)
+				)
+				(justify right)
+			)
+		)
+		(pin "LOAD1_3V3" output
+			(at 120.65 105.41 0)
+			(effects
+				(font
+					(size 1.27 1.27)
+				)
+				(justify right)
+			)
+		)
+		(pin "LOAD2_EN" input
+			(at 87.63 107.95 180)
+			(effects
+				(font
+					(size 1.27 1.27)
+				)
+				(justify left)
+			)
+		)
+		(pin "LOAD1_EN" input
+			(at 87.63 105.41 180)
+			(effects
+				(font
+					(size 1.27 1.27)
+				)
+				(justify left)
+			)
+		)
