File: LoRaNode328.kicad_sch (KiCad schematic)
At the start: 0 parts

Commit message: jst
Other:
- sheet Connectors: file Connectors.kicad_sch -> ./schematics/Connectors.kicad_sch
- sheet Connectors ports: added BAT+, BAT-; removed none
- sheet LoRa: file LoRa.kicad_sch -> ./schematics/LoRa.kicad_sch
- sheet MCU: file MCU.kicad_sch -> ./schematics/MCU.kicad_sch
- sheet Power_Control: file Power_Control.kicad_sch -> ./schematics/Power_Control.kicad_sch
- sheet Power_Regulator: file Power_Regulator.sch.kicad_sch -> ./schematics/Power_Regulator.sch.kicad_sch
- sheet Sensors: file Sensors.kicad_sch -> ./schematics/Sensors.kicad_sch
Changed lines of the file:
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@@
 			)
 		)
-		(property "Sheetfile" "LoRa.kicad_sch"
+		(property "Sheetfile" "./schematics/LoRa.kicad_sch"
 			(at 87.63 59.0046 0)
 			(effects
@@
 		)
 		(pin "LORA_3V3" input
-			(at 87.63 35.56 180)
+			(at 87.63 33.02 180)
 			(effects
 				(font
@@
 		)
 		(pin "RAK_PB12" output
-			(at 119.38 43.18 0)
+			(at 119.38 40.64 0)
 			(effects
 				(font
@@
 		)
 		(pin "RAK_PA1" output
+			(at 119.38 35.56 0)
+			(effects
+				(font
+					(size 1.27 1.27)
+				)
+				(justify right)
+			)
+		)
+		(pin "RAK_PB5" output
 			(at 119.38 38.1 0)
 			(effects
@@
 			)
 		)
-		(pin "RAK_PB5" output
-			(at 119.38 40.64 0)
-			(effects
-				(font
-					(size 1.27 1.27)
-				)
-				(justify right)
-			)
-		)
 		(pin "RAK_PA0" output
-			(at 119.38 35.56 0)
+			(at 119.38 33.02 0)
 			(effects
 				(font
@@
 		)
 		(pin "RAK_RESET" input
+			(at 87.63 36.83 180)
+			(effects
+				(font
+					(size 1.27 1.27)
+				)
+				(justify left)
+			)
+		)
+		(pin "RAK_UART1_RX" input
+			(at 87.63 43.18 180)
+			(effects
+				(font
+					(size 1.27 1.27)
+				)
+				(justify left)
+			)
+		)
+		(pin "RAK_UART1_TX" output
+			(at 87.63 45.72 180)
+			(effects
+				(font
+					(size 1.27 1.27)
+				)
+				(justify left)
+			)
+		)
+		(pin "RAK_BOOT" input
 			(at 87.63 39.37 180)
 			(effects
@@
 			)
 		)
-		(pin "RAK_UART1_RX" input
-			(at 87.63 45.72 180)
-			(effects
-				(font
-					(size 1.27 1.27)
-				)
-				(justify left)
-			)
-		)
-		(pin "RAK_UART1_TX" output
-			(at 87.63 48.26 180)
-			(effects
-				(font
-					(size 1.27 1.27)
-				)
-				(justify left)
-			)
-		)
-		(pin "RAK_BOOT" input
-			(at 87.63 41.91 180)
-			(effects
-				(font
-					(size 1.27 1.27)
-				)
-				(justify left)
-			)
-		)
 		(pin "RAK_UART2_TX" output
-			(at 87.63 54.61 180)
+			(at 87.63 52.07 180)
 			(effects
 				(font
@@
 		)
 		(pin "RAK_UART2_RX" input
-			(at 87.63 52.07 180)
+			(at 87.63 49.53 180)
 			(effects
 				(font
@@
 			)
 		)
-		(property "Sheetfile" "Power_Regulator.sch.kicad_sch"
+		(property "Sheetfile" "./schematics/Power_Regulator.sch.kicad_sch"
 			(at 35.56 41.2246 0)
 			(effects
@@
 		)
 		(pin "VCC_3V3" output
-			(at 71.12 35.56 0)
+			(at 71.12 33.02 0)
 			(effects
 				(font
@@
 		)
 		(pin "VBAT" input
-			(at 35.56 35.56 180)
+			(at 35.56 33.02 180)
 			(effects
 				(font
@@
 			)
 		)
-		(property "Sheetfile" "Sensors.kicad_sch"
+		(property "Sheetfile" "./schematics/Sensors.kicad_sch"
 			(at 88.9 83.1346 0)
 			(effects
@@
 	(sheet
 		(at 132.08 30.48)
-		(size 12.7 5.08)
+		(size 31.75 7.62)
 		(fields_autoplaced yes)
 		(stroke
@@
 			)
 		)
-		(property "Sheetfile" "Connectors.kicad_sch"
-			(at 132.08 36.1446 0)
+		(property "Sheetfile" "./schematics/Connectors.kicad_sch"
+			(at 132.08 38.6846 0)
 			(effects
 				(font
@@
 				)
 				(justify left top)
+			)
+		)
+		(pin "BAT+" output
+			(at 163.83 33.02 0)
+			(effects
+				(font
+					(size 1.27 1.27)
+				)
+				(justify right)
+			)
+		)
+		(pin "BAT-" output
+			(at 163.83 35.56 0)
+			(effects
+				(font
+					(size 1.27 1.27)
+				)
+				(justify right)
 			)
 		)
@@
 			)
 		)
-		(property "Sheetfile" "MCU.kicad_sch"
+		(property "Sheetfile" "./schematics/MCU.kicad_sch"
 			(at 35.56 102.1846 0)
 			(effects
@@
 			)
 		)
-		(property "Sheetfile" "Power_Control.kicad_sch"
+		(property "Sheetfile" "./schematics/Power_Control.kicad_sch"
 			(at 87.63 114.8846 0)
 			(effects

Commit message: Connectors
Other:
- sheet Connectors ports: added 3V3+, 3V3-, FTDI_DTR, FTDI_RX, FTDI_TX, FTDI_VCC, I2C_SCL, I2C_SDA, I2C_VCC, ISP_MISO, ISP_MOSI, ISP_RESET, ISP_SCK, ISP_VCC, LOAD1+, LOAD1-, LOAD2+, LOAD2-, LORA_UART1_RX, LORA_UART1_TX, LORA_UART2_RX, LORA_UART2_TX, LORA_VCC, SENS_SCL, SENS_SDA, SENS_VCC, SPI_MISO, SPI_MOSI, SPI_SCK, SPI_SS, UART1_RX, UART1_TX, UART1_VCC; removed none

Commit message: root scheme
Other:
- sheet Connectors ports: added none; removed 3V3-, ISP_VCC, LOAD1-, LOAD2-
- sheet MCU ports: added LOADX2_EN, LOADX_EN, LORA_EN, SCL, SDA, SENS_EN; removed LOAD4_EN, RF95W_EN, RF_PWR_EN, SCL_L, SDA_L
- sheet Power_Control ports: added PWR_C_3V3; removed LC_3V3
- sheet Power_Regulator ports: added VBAT+, VBAT-; removed VBAT

Commit message: connectors
Other:
- sheet Connectors ports: added LORA_BOOT, LORA_RESET; removed FTDI_VCC, I2C_VCC, SENS_VCC, UART1_VCC
- sheet LoRa ports: added none; removed RAK_PA0, RAK_PA1, RAK_PB12, RAK_PB5
- sheet MCU ports: added LORA_RX, LORA_TX, SPI_SS; removed BAT_CHARGE, LOADX2_EN, LOADX_EN, RF95W_DIO0, RF95W_DIO1, RF95W_DIO2, RF_RX_L, RF_TX_L, WD_DONE
- note added: "IMPORTANTE: Los pines ICP (ISP) y FTDI son para programación sin fuente. Para comunicación con el sistema alimentado, NO conectar VCC del FTDI."

Commit message: ERC
Other:
- sheet Connectors ports: added none; removed BAT-
- sheet Power_Regulator ports: added none; removed VBAT-
Changed lines of the file:
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@@
-	(wire
-		(pts
-			(xy 78.74 81.28) (xy 78.74 129.54)
-		)
-		(stroke
-			(width 0)
-			(type default)
-		)
-	)
 	(wire
 		(pts
@@
 	(wire
 		(pts
-			(xy 81.28 81.28) (xy 81.28 129.54)
-		)
-		(stroke
-			(width 0)
-			(type default)
-		)
-	)
-	(wire
-		(pts
 			(xy 175.26 124.46) (xy 175.26 129.54)
 		)
@@
 		(pts
 			(xy 160.02 71.12) (xy 177.8 71.12)
+		)
+		(stroke
+			(width 0)
+			(type default)
+		)
+	)
+	(wire
+		(pts
+			(xy 78.74 78.74) (xy 78.74 129.54)
 		)
 		(stroke
@@
 	)
 	(sheet
-		(at 73.66 63.5)
-		(size 20.32 17.78)
+		(at 76.2 63.5)
+		(size 17.78 15.24)
 		(fields_autoplaced yes)
 		(stroke
@@
 		)
 		(property "Sheetname" "Power_Regulator"
-			(at 73.66 62.7884 0)
+			(at 76.2 62.7884 0)
 			(effects
 				(font
@@
 		)
 		(property "Sheetfile" "./schematics/Power_Regulator.sch.kicad_sch"
-			(at 73.66 81.8646 0)
+			(at 76.2 79.3246 0)
 			(effects
 				(font
@@
 		)
 		(pin "VBAT+" input
-			(at 78.74 81.28 270)
-			(effects
-				(font
-					(size 1.27 1.27)
-				)
-				(justify left)
-			)
-		)
-		(pin "VBAT-" input
-			(at 81.28 81.28 270)
+			(at 78.74 78.74 270)
 			(effects
 				(font
@@
 			)
 		)
-		(pin "BAT-" input
-			(at 81.28 129.54 90)
-			(effects
-				(font
-					(size 1.27 1.27)
-				)
-				(justify right)
-			)
-		)
-		(pin "BAT+" input
-			(at 78.74 129.54 90)
-			(effects
-				(font
-					(size 1.27 1.27)
-				)
-				(justify right)
-			)
-		)
 		(pin "ISP_MOSI" output
 			(at 115.57 129.54 90)
@@
 			(effects
 				(font
+					(size 1.27 1.27)
+				)
+				(justify right)
+			)
+		)
+		(pin "BAT+" output
+			(at 78.74 129.54 90)
+			(effects
+				(font
