File: Power_Control.kicad_sch (KiCad schematic)
At the start: 0 parts

Commit message: load control
Parts:
- added C15, C17, C19, C21, C23, C24, C27, C28: 0.1uF, symbol Device:C_Small
- added C16, C18, C20, C22, C25, C26, C29, C30: 10uF, symbol Device:C_Small
- added U5, U6, U7, U8: AP2171W, Package_TO_SOT_SMD:SOT-23-5, symbol Power_Management:AP2171W
Connections:
- new net GND: C15.2, C16.2, C17.2, C18.2, C19.2, C20.2, C21.2, C22.2, C23.2, C24.2, C25.2, C26.2, C27.2, C28.2, C29.2, C30.2, U5.2 (GND), U6.2 (GND), U7.2 (GND), U8.2 (GND)
- new net LC_3V3: C17.1, C18.1, C19.1, C20.1, C23.1, C24.1, C25.1, C26.1, U5.5 (IN), U6.5 (IN), U7.5 (IN), U8.5 (IN)
- new net LOAD1_3V3: C27.1, C29.1, U7.1 (OUT)
- new net LOAD1_EN: U7.4 (EN)
- new net LOAD2_3V3: C28.1, C30.1, U8.1 (OUT)
- new net LOAD2_EN: U8.4 (EN)
- new net LORA_3V3: C15.1, C16.1, U5.1 (OUT)
- new net LORA_EN: U5.4 (EN)
- new net SENS_3V3: C21.1, C22.1, U6.1 (OUT)
- new net SENS_EN: U6.4 (EN)
- no-connect marks 0 -> 4
