File: schematics/Connectors.kicad_sch (KiCad schematic)
At the start: 1 part, among them J1 B2B-XH-A__LF__SN_

Commit message: Connectors
Parts:
- added J10: SPI, symbol Connector_Generic:Conn_01x04
- added J11: ISP, symbol Connector_Generic:Conn_02x03_Odd_Even
- added J2: FTDI, symbol Connector_Generic:Conn_01x06
- added J3: UART, symbol Connector_Generic:Conn_01x06
- added J4: I2C, symbol Connector_Generic:Conn_01x04
- added J5: LORA, symbol Connector_Generic:Conn_01x06
- added J6: SENSOR, symbol Connector_Generic:Conn_01x04
- added J7: LOAD1, B2B-XH-A__LF__SN_:JST_B2B-XH-A__LF__SN_, symbol B2B-XH-A__LF__SN_:B2B-XH-A__LF__SN_
- added J8: LOAD2, B2B-XH-A__LF__SN_:JST_B2B-XH-A__LF__SN_, symbol B2B-XH-A__LF__SN_:B2B-XH-A__LF__SN_
- added J9: 3V3, B2B-XH-A__LF__SN_:JST_B2B-XH-A__LF__SN_, symbol B2B-XH-A__LF__SN_:B2B-XH-A__LF__SN_
- J1: value B2B-XH-A__LF__SN_ -> BAT
Connections:
- new net 3V3+: J9.1
- new net 3V3-: J9.2
- new net FTDI_DTR: J2.1 (Pin_1)
- new net FTDI_RX: J2.2 (Pin_2)
- new net FTDI_TX: J2.3 (Pin_3)
- new net FTDI_VCC: J2.4 (Pin_4)
- new net GND: J11.6 (Pin_6), J2.6 (Pin_6), J3.1 (Pin_1), J4.1 (Pin_1), J5.1 (Pin_1), J6.1 (Pin_1)
- new net I2C_SCL: J4.4 (Pin_4)
- new net I2C_SDA: J4.3 (Pin_3)
- new net I2C_VCC: J4.2 (Pin_2)
- new net ISP_MISO: J11.1 (Pin_1)
- new net ISP_MOSI: J11.4 (Pin_4)
- new net ISP_RESET: J11.5 (Pin_5)
- new net ISP_SCK: J11.3 (Pin_3)
- new net ISP_VCC: J11.2 (Pin_2)
- new net LOAD1+: J7.1
- new net LOAD1-: J7.2
- new net LOAD2+: J8.1
- new net LOAD2-: J8.2
- new net LORA_UART1_RX: J5.4 (Pin_4)
- new net LORA_UART1_TX: J5.3 (Pin_3)
- new net LORA_UART2_RX: J5.6 (Pin_6)
- new net LORA_UART2_TX: J5.5 (Pin_5)
- new net LORA_VCC: J5.2 (Pin_2)
- new net SENS_SCL: J6.4 (Pin_4)
- new net SENS_SDA: J6.3 (Pin_3)
- new net SENS_VCC: J6.2 (Pin_2)
- new net SPI_MISO: J10.1 (Pin_1)
- new net SPI_MOSI: J10.2 (Pin_2)
- new net SPI_SCK: J10.3 (Pin_3)
- new net SPI_SS: J10.4 (Pin_4)
- new net UART1_RX: J3.5 (Pin_5)
- new net UART1_TX: J3.4 (Pin_4)
- new net UART1_VCC: J3.3 (Pin_3)
- no-connect marks 0 -> 3
Other:
- moved on the sheet: J1

Commit message: root scheme
Connections:
- net 3V3- is gone; now on net GND: J9.2
- net ISP_VCC is gone; now on net 3V3+: J11.2 (Pin_2)
- net LOAD1- is gone; now on net GND: J7.2
- net LOAD2- is gone; now on net GND: J8.2
- net FTDI_VCC: no longer names the net of J2.4 (Pin_4)
Changed lines of the file:
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@@
+		)
+	)
+	(hierarchical_label "3V3+"
+		(shape output)
+		(at 106.68 55.88 0)
+		(fields_autoplaced yes)
+		(effects
+			(font
+				(size 1.27 1.27)
+			)
+			(justify left)
 		)
 	)
@@
 		)
 	)
-	(hierarchical_label "LOAD1-"
-		(shape output)
-		(at 180.34 59.69 180)
-		(fields_autoplaced yes)
-		(effects
-			(font
-				(size 1.27 1.27)
-			)
-			(justify right)
-		)
-	)
 	(hierarchical_label "I2C_SDA"
 		(shape bidirectional)
@@
 		)
 	)
-	(hierarchical_label "LOAD2-"
-		(shape output)
-		(at 180.34 73.66 180)
-		(fields_autoplaced yes)
-		(effects
-			(font
-				(size 1.27 1.27)
-			)
-			(justify right)
-		)
-	)
 	(hierarchical_label "UART1_RX"
 		(shape input)
@@
 		)
 	)
-	(hierarchical_label "3V3-"
-		(shape output)
-		(at 180.34 45.72 180)
-		(fields_autoplaced yes)
-		(effects
-			(font
-				(size 1.27 1.27)
-			)
-			(justify right)
-		)
-	)
 	(hierarchical_label "I2C_VCC"
 		(shape output)
@@
 		(shape input)
 		(at 127 43.18 180)
-		(fields_autoplaced yes)
-		(effects
-			(font
-				(size 1.27 1.27)
-			)
-			(justify right)
-		)
-	)
-	(hierarchical_label "ISP_VCC"
-		(shape input)
-		(at 106.68 55.88 0)
-		(fields_autoplaced yes)
-		(effects
-			(font
-				(size 1.27 1.27)
-			)
-			(justify left)
-		)
-	)
-	(hierarchical_label "FTDI_VCC"
-		(shape input)
-		(at 132.08 63.5 180)
 		(fields_autoplaced yes)
 		(effects
@@
 	(symbol
 		(lib_id "power:GND")
+		(at 180.34 59.69 0)
+		(unit 1)
+		(exclude_from_sim no)
+		(in_bom yes)
+		(on_board yes)
+		(dnp no)
+		(fields_autoplaced yes)
+		(property "Reference" "#PWR049"
+			(at 180.34 66.04 0)
+			(effects
+				(font
+					(size 1.27 1.27)
+				)
+				(hide yes)
+			)
+		)
+		(property "Value" "GND"
+			(at 180.34 64.77 0)
+			(effects
+				(font
+					(size 1.27 1.27)
+				)
+			)
+		)
+		(property "Footprint" ""
+			(at 180.34 59.69 0)
+			(effects
+				(font
+					(size 1.27 1.27)
+				)
+				(hide yes)
+			)
+		)
+		(property "Datasheet" ""
+			(at 180.34 59.69 0)
+			(effects
+				(font
+					(size 1.27 1.27)
+				)
+				(hide yes)
+			)
+		)
+		(property "Description" "Power symbol creates a global label with name \"GND\" , ground"
+			(at 180.34 59.69 0)
+			(effects
+				(font
+					(size 1.27 1.27)
+				)
+				(hide yes)
+			)
+		)
+		(pin "1"
+		)
+		(instances
+			(project "LoRaNode328"
+				(path "/e0ffc31c-24f5-4303-8af9-d0625c9ddd62/c4f9c729-ac2e-4c38-94d3-26bb33a7c408"
+					(reference "#PWR049")
+					(unit 1)
+				)
+			)
+		)
+	)
+	(symbol
+		(lib_id "power:GND")
 		(at 106.68 60.96 0)
 		(unit 1)
@@
 				(path "/e0ffc31c-24f5-4303-8af9-d0625c9ddd62/c4f9c729-ac2e-4c38-94d3-26bb33a7c408"
 					(reference "J6")
+					(unit 1)
+				)
+			)
+		)
+	)
+	(symbol
+		(lib_id "power:GND")
+		(at 180.34 73.66 0)
+		(unit 1)
+		(exclude_from_sim no)
+		(in_bom yes)
+		(on_board yes)
+		(dnp no)
+		(fields_autoplaced yes)
+		(property "Reference" "#PWR050"
+			(at 180.34 80.01 0)
+			(effects
+				(font
+					(size 1.27 1.27)
+				)
+				(hide yes)
+			)
+		)
+		(property "Value" "GND"
+			(at 180.34 78.74 0)
+			(effects
+				(font
+					(size 1.27 1.27)
+				)
+			)
+		)
+		(property "Footprint" ""
+			(at 180.34 73.66 0)
+			(effects
+				(font
+					(size 1.27 1.27)
+				)
+				(hide yes)
+			)
+		)
+		(property "Datasheet" ""
+			(at 180.34 73.66 0)
+			(effects
+				(font
+					(size 1.27 1.27)
+				)
+				(hide yes)
+			)
+		)
+		(property "Description" "Power symbol creates a global label with name \"GND\" , ground"
+			(at 180.34 73.66 0)
+			(effects
+				(font
+					(size 1.27 1.27)
+				)
+				(hide yes)
+			)
+		)
+		(pin "1"
+		)
+		(instances
+			(project "LoRaNode328"
+				(path "/e0ffc31c-24f5-4303-8af9-d0625c9ddd62/c4f9c729-ac2e-4c38-94d3-26bb33a7c408"
+					(reference "#PWR050")
 					(unit 1)
 				)
@@
 					(unit 1)
 				)
+			)
+		)
+	)
+	(symbol
+		(lib_id "power:GND")
+		(at 180.34 45.72 0)
+		(unit 1)
+		(exclude_from_sim no)
+		(in_bom yes)
+		(on_board yes)
+		(dnp no)
+		(fields_autoplaced yes)
+		(property "Reference" "#PWR048"
+			(at 180.34 52.07 0)
+			(effects
+				(font
+					(size 1.27 1.27)
+				)
+				(hide yes)
+			)
+		)
+		(property "Value" "GND"
+			(at 180.34 50.8 0)
+			(effects
+				(font
+					(size 1.27 1.27)
+				)
+			)
+		)
+		(property "Footprint" ""
+			(at 180.34 45.72 0)
+			(effects
+				(font
+					(size 1.27 1.27)
+				)
+				(hide yes)
+			)
+		)
+		(property "Datasheet" ""
+			(at 180.34 45.72 0)
+			(effects
+				(font
+					(size 1.27 1.27)
+				)
+				(hide yes)
+			)
+		)
+		(property "Description" "Power symbol creates a global label with name \"GND\" , ground"
+			(at 180.34 45.72 0)
+			(effects
+				(font
+					(size 1.27 1.27)
+				)
+				(hide yes)
+			)
+		)
+		(pin "1"
+		)
+		(instances
+			(project "LoRaNode328"
+				(path "/e0ffc31c-24f5-4303-8af9-d0625c9ddd62/c4f9c729-ac2e-4c38-94d3-26bb33a7c408"
+					(reference "#PWR048")
+					(unit 1)
+				)

Commit message: connectors
Parts:
- removed J5: LORA, symbol Connector_Generic:Conn_01x06
- added J12: LORA, symbol Connector_Generic:Conn_01x08
Connections:
- net I2C_VCC is gone; now on net 3V3+: J4.2 (Pin_2)
- net SENS_VCC is gone; now on net 3V3+: J6.2 (Pin_2)
- net UART1_VCC is gone; now on net 3V3+: J3.3 (Pin_3)
- net 3V3+: now also J2.4 (Pin_4)
- net GND: now also J12.1 (Pin_1)
- net LORA_UART1_RX: now also J12.4 (Pin_4)
- net LORA_UART1_TX: now also J12.3 (Pin_3)
- net LORA_UART2_RX: now also J12.6 (Pin_6)
- net LORA_UART2_TX: now also J12.5 (Pin_5)
- net LORA_VCC: now also J12.2 (Pin_2)
- new net LORA_BOOT: J12.7 (Pin_7)
- new net LORA_RESET: J12.8 (Pin_8)
Other:
- note added: "IMPORTANTE: Los pines ICP (ISP) y FTDI son para programación sin fuente. Para comunicación con el sistema alimentado, NO conectar VCC del FTDI."

Commit message: ERC
Parts:
- J1: value BAT -> 3V3
Connections:
- net BAT- is gone; now on net GND: J1.2
Other:
- moved on the sheet: J11, J2
