File: schematics/LoRa.kicad_sch (KiCad schematic)
At the start: 10 parts, among them SW1 SW_Push, SW2 SW_Push, U3 RAK3172

Commit message: connectors
Parts:
- removed D2: LED_Small, symbol Device:LED_Small
- removed R4: 4K7, symbol Device:R_Small
Connections:
- net RAK_PA0: no longer names the net of U3.29 (PA0)
- net RAK_PA1: no longer names the net of U3.6 (PA1)
- net RAK_PB12: no longer names the net of U3.27 (PB12)
- net RAK_PB5: no longer names the net of U3.30 (PB5)
- no-connect marks 16 -> 20

Commit message: ERC
Parts:
- U3: footprint (none) -> RAK3172:RAK3172
Changed lines of the file:
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@@
 			)
 		)
-		(property "Footprint" ""
+		(property "Footprint" "RAK3172:RAK3172"
 			(at 132.08 64.77 0)
 			(effects
