File: schematics/MCU.kicad_sch (KiCad schematic)
At the start: 10 parts, among them U2 ATmega328P-A, Y2 8MHz

Commit message: root scheme
Connections:
- net LOAD2_EN: no longer U2.13 (PB1)
- net LOAD4_EN renamed LOADX2_EN
- net RF95W_EN renamed LOADX_EN
- net RF_PWR_EN renamed LORA_EN
- net SCL_L renamed SCL
- net SDA_L renamed SDA
- new net SENS_EN: U2.13 (PB1)
Changed lines of the file:
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@@
 		)
 	)
-	(hierarchical_label "LOAD2_EN"
+	(hierarchical_label "SENS_EN"
 		(shape output)
 		(at 165.1 68.58 0)
@@
 		)
 	)
-	(hierarchical_label "RF95W_EN"
+	(hierarchical_label "LOADX_EN"
 		(shape output)
 		(at 165.1 71.12 0)
@@
 		)
 	)
-	(hierarchical_label "SCL_L"
+	(hierarchical_label "SCL"
 		(shape output)
 		(at 165.1 101.6 0)
@@
 		)
 	)
-	(hierarchical_label "SDA_L"
+	(hierarchical_label "SDA"
 		(shape output)
 		(at 165.1 99.06 0)
@@
 		)
 	)
-	(hierarchical_label "RF_PWR_EN"
+	(hierarchical_label "LORA_EN"
 		(shape output)
 		(at 165.1 66.04 0)
@@
 		)
 	)
-	(hierarchical_label "LOAD4_EN"
+	(hierarchical_label "LOADX2_EN"
 		(shape output)
 		(at 165.1 127 0)

Commit message: connectors
Connections:
- net BAT_CHARGE: no longer names the net of U2.19 (ADC6)
- net LOADX2_EN: no longer names the net of U2.11 (PD7)
- net LOADX_EN renamed SPI_SS
- net RF95W_DIO0: no longer names the net of U2.32 (PD2)
- net RF95W_DIO1: no longer names the net of U2.1 (PD3)
- net RF95W_DIO2: no longer names the net of U2.2 (PD4)
- net RF_RX_L renamed LORA_RX
- net RF_TX_L renamed LORA_TX
- net WD_DONE: no longer names the net of U2.23 (PC0)
- no-connect marks 2 -> 8
Changed lines of the file:
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@@
+	)
+	(no_connect
+		(at 158.75 119.38)
 	)
 	(no_connect
 		(at 128.27 73.66)
 	)
-	(wire
-		(pts
-			(xy 158.75 116.84) (xy 165.1 116.84)
+	(no_connect
+		(at 128.27 71.12)
+	)
+	(no_connect
+		(at 158.75 88.9)
+	)
+	(no_connect
+		(at 158.75 127)
+	)
+	(no_connect
+		(at 158.75 116.84)
+	)
+	(no_connect
+		(at 158.75 114.3)
+	)
+	(wire
+		(pts
+			(xy 158.75 71.12) (xy 165.1 71.12)
 		)
 		(stroke
@@
 	(wire
 		(pts
-			(xy 158.75 88.9) (xy 165.1 88.9)
-		)
-		(stroke
-			(width 0)
-			(type default)
-		)
-	)
-	(wire
-		(pts
 			(xy 171.45 45.72) (xy 171.45 48.26)
 		)
@@
 	(wire
 		(pts
-			(xy 158.75 71.12) (xy 165.1 71.12)
-		)
-		(stroke
-			(width 0)
-			(type default)
-		)
-	)
-	(wire
-		(pts
 			(xy 158.75 83.82) (xy 189.23 83.82)
 		)
@@
 	(wire
 		(pts
-			(xy 111.76 71.12) (xy 128.27 71.12)
-		)
-		(stroke
-			(width 0)
-			(type default)
-		)
-	)
-	(wire
-		(pts
-			(xy 158.75 127) (xy 165.1 127)
-		)
-		(stroke
-			(width 0)
-			(type default)
-		)
-	)
-	(wire
-		(pts
 			(xy 158.75 111.76) (xy 165.1 111.76)
 		)
@@
 	(wire
 		(pts
-			(xy 111.76 68.58) (xy 111.76 71.12)
-		)
-		(stroke
-			(width 0)
-			(type default)
-		)
-	)
-	(wire
-		(pts
 			(xy 158.75 66.04) (xy 165.1 66.04)
 		)
@@
 	(wire
 		(pts
-			(xy 158.75 114.3) (xy 165.1 114.3)
-		)
-		(stroke
-			(width 0)
-			(type default)
-		)
-	)
-	(wire
-		(pts
 			(xy 99.06 66.04) (xy 99.06 68.58)
 		)
@@
 	(wire
 		(pts
-			(xy 158.75 119.38) (xy 165.1 119.38)
-		)
-		(stroke
-			(width 0)
-			(type default)
-		)
-	)
-	(wire
-		(pts
 			(xy 171.45 38.1) (xy 161.29 38.1)
 		)
@@
 	)
 	(hierarchical_label "DTR"
-		(shape output)
+		(shape input)
 		(at 190.5 125.73 0)
 		(fields_autoplaced yes)
@@
 		)
 	)
-	(hierarchical_label "WD_DONE"
-		(shape output)
-		(at 165.1 88.9 0)
-		(fields_autoplaced yes)
-		(effects
-			(font
-				(size 1.27 1.27)
-			)
-			(justify left)
-		)
-	)
 	(hierarchical_label "SENS_EN"
 		(shape output)
@@
 		)
 	)
-	(hierarchical_label "LOADX_EN"
-		(shape output)
-		(at 165.1 71.12 0)
-		(fields_autoplaced yes)
-		(effects
-			(font
-				(size 1.27 1.27)
-			)
-			(justify left)
-		)
-	)
-	(hierarchical_label "BAT_CHARGE"
+	(hierarchical_label "SCL"
+		(shape output)
+		(at 165.1 101.6 0)
+		(fields_autoplaced yes)
+		(effects
+			(font
+				(size 1.27 1.27)
+			)
+			(justify left)
+		)
+	)
+	(hierarchical_label "SDA"
+		(shape bidirectional)
+		(at 165.1 99.06 0)
+		(fields_autoplaced yes)
+		(effects
+			(font
+				(size 1.27 1.27)
+			)
+			(justify left)
+		)
+	)
+	(hierarchical_label "SPI_MISO"
 		(shape input)
-		(at 111.76 68.58 0)
-		(fields_autoplaced yes)
-		(effects
-			(font
-				(size 1.27 1.27)
-			)
-			(justify left)
-		)
-	)
-	(hierarchical_label "SCL"
-		(shape output)
-		(at 165.1 101.6 0)
-		(fields_autoplaced yes)
-		(effects
-			(font
-				(size 1.27 1.27)
-			)
-			(justify left)
-		)
-	)
-	(hierarchical_label "SDA"
-		(shape output)
-		(at 165.1 99.06 0)
-		(fields_autoplaced yes)
-		(effects
-			(font
-				(size 1.27 1.27)
-			)
-			(justify left)
-		)
-	)
-	(hierarchical_label "SPI_MISO"
-		(shape output)
 		(at 165.1 76.2 0)
 		(fields_autoplaced yes)
@@
 		)
 	)
-	(hierarchical_label "RF95W_DIO1"
-		(shape output)
-		(at 165.1 116.84 0)
-		(fields_autoplaced yes)
-		(effects
-			(font
-				(size 1.27 1.27)
-			)
-			(justify left)
-		)
-	)
 	(hierarchical_label "SPI_SCLK"
 		(shape output)
 		(at 165.1 78.74 0)
-		(fields_autoplaced yes)
-		(effects
-			(font
-				(size 1.27 1.27)
-			)
-			(justify left)
-		)
-	)
-	(hierarchical_label "RF95W_DIO2"
-		(shape output)
-		(at 165.1 119.38 0)
 		(fields_autoplaced yes)
 		(effects
@@
 		)
 	)
-	(hierarchical_label "RF_TX_L"
-		(shape output)
+	(hierarchical_label "LORA_TX"
+		(shape input)
 		(at 165.1 124.46 0)
 		(fields_autoplaced yes)
@@
 	)
 	(hierarchical_label "RXI"
-		(shape output)
+		(shape input)
 		(at 165.1 109.22 0)
 		(fields_autoplaced yes)
@@
 		)
 	)
-	(hierarchical_label "LOADX2_EN"
-		(shape output)
-		(at 165.1 127 0)
-		(fields_autoplaced yes)
-		(effects
-			(font
-				(size 1.27 1.27)
-			)
-			(justify left)
-		)
-	)
-	(hierarchical_label "RF_RX_L"
+	(hierarchical_label "LORA_RX"
 		(shape output)
 		(at 165.1 121.92 0)
@@
 		)
 	)
+	(hierarchical_label "SPI_SS"
+		(shape output)
+		(at 165.1 71.12 0)
+		(fields_autoplaced yes)
+		(effects
+			(font
+				(size 1.27 1.27)
+			)
+			(justify left)
+		)
+	)
 	(hierarchical_label "LOAD1_EN"
 		(shape output)
@@
 		(fields_autoplaced yes)
 		(effects
-			(font
-				(size 1.27 1.27)
-			)
-			(justify left)
-		)
-	)
-	(hierarchical_label "RF95W_DIO0"
-		(shape output)
-		(at 165.1 114.3 0)
-		(fields_autoplaced yes)
-		(effects

Commit message: ERC
Changed lines of the file:
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@@
+	)
+	(junction
+		(at 171.45 38.1)
+		(diameter 0)
+		(color 0 0 0 0)
 	)
 	(junction
@@
 					(unit 1)
 				)
+			)
+		)
+	)
+	(symbol
+		(lib_id "power:PWR_FLAG")
+		(at 171.45 38.1 0)
+		(unit 1)
+		(exclude_from_sim no)
+		(in_bom yes)
+		(on_board yes)
+		(dnp no)
+		(fields_autoplaced yes)
+		(property "Reference" "#FLG03"
+			(at 171.45 36.195 0)
+			(effects
+				(font
+					(size 1.27 1.27)
+				)
+				(hide yes)
+			)
+		)
+		(property "Value" "PWR_FLAG"
+			(at 171.45 33.02 0)
+			(effects
+				(font
+					(size 1.27 1.27)
+				)
+			)
+		)
+		(property "Footprint" ""
+			(at 171.45 38.1 0)
+			(effects
+				(font
+					(size 1.27 1.27)
+				)
+				(hide yes)
+			)
+		)
+		(property "Datasheet" "~"
+			(at 171.45 38.1 0)
+			(effects
+				(font
+					(size 1.27 1.27)
+				)
+				(hide yes)
+			)
+		)
+		(property "Description" "Special symbol for telling ERC where power comes from"
+			(at 171.45 38.1 0)
+			(effects
+				(font
+					(size 1.27 1.27)
+				)
+				(hide yes)
+			)
+		)
+		(pin "1"
+		)
+		(instances
+			(project ""
+				(path "/e0ffc31c-24f5-4303-8af9-d0625c9ddd62/c544bbb4-4120-4a0c-b3e8-54718c20e48f"
+					(reference "#FLG03")
+					(unit 1)
+				)
