File: schematics/Power_Control.kicad_sch (KiCad schematic)
At the start: 20 parts, among them U5 AP2171W, U6 AP2171W, U7 AP2171W, U8 AP2171W

Commit message: root scheme
Connections:
- net LC_3V3 renamed PWR_C_3V3
Changed lines of the file:
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@@
 		)
 	)
-	(hierarchical_label "LC_3V3"
+	(hierarchical_label "PWR_C_3V3"
 		(shape input)
 		(at 87.63 30.48 180)
@@
 		)
 	)
-	(hierarchical_label "LC_3V3"
+	(hierarchical_label "PWR_C_3V3"
 		(shape input)
 		(at 87.63 104.14 180)
@@
 		)
 	)
-	(hierarchical_label "LC_3V3"
+	(hierarchical_label "PWR_C_3V3"
 		(shape input)
 		(at 87.63 66.04 180)
@@
 		)
 	)
-	(hierarchical_label "LC_3V3"
+	(hierarchical_label "PWR_C_3V3"
 		(shape input)
 		(at 87.63 139.7 180)

Commit message: connectors
Parts:
- added D2, D3, D4, D5: LED_Small, symbol Device:LED_Small
- added R4, R7, R8, R9: 4K7, symbol Device:R_Small
Connections:
- net GND: now also D2.1 (K), D3.1 (K), D4.1 (K), D5.1 (K)
- net LOAD1_3V3: now also R8.1
- net LOAD2_3V3: now also R9.1
- net LORA_3V3: now also R4.1
- net SENS_3V3: now also R7.1
- new net: D2.2 (A), R4.2
- new net: D5.2 (A), R9.2
- new net: D3.2 (A), R7.2
- new net: D4.2 (A), R8.2

Commit message: ERC
Parts:
- removed D2: LED_Small, symbol Device:LED_Small
- removed R4: 4K7, symbol Device:R_Small
Changed lines of the file:
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@@
 	(wire
 		(pts
-			(xy 193.04 38.1) (xy 193.04 40.64)
-		)
-		(stroke
-			(width 0)
-			(type default)
-		)
-	)
-	(wire
-		(pts
 			(xy 172.72 139.7) (xy 176.53 139.7)
 		)
@@
 	(wire
 		(pts
-			(xy 193.04 30.48) (xy 193.04 33.02)
-		)
-		(stroke
-			(width 0)
-			(type default)
-		)
-	)
-	(wire
-		(pts
 			(xy 87.63 139.7) (xy 92.71 139.7)
 		)
@@
 	(wire
 		(pts
-			(xy 193.04 45.72) (xy 193.04 48.26)
-		)
-		(stroke
-			(width 0)
-			(type default)
-		)
-	)
-	(wire
-		(pts
 			(xy 152.4 139.7) (xy 161.29 139.7)
 		)
@@
 		)
 	)
-	(hierarchical_label "LORA_3V3"
-		(shape output)
-		(at 193.04 30.48 0)
-		(fields_autoplaced yes)
-		(effects
-			(font
-				(size 1.27 1.27)
-			)
-			(justify left)
-		)
-	)
 	(hierarchical_label "LOAD1_3V3"
 		(shape output)
@@
 	)
 	(symbol
-		(lib_id "Device:LED_Small")
-		(at 193.04 43.18 90)
-		(unit 1)
-		(exclude_from_sim no)
-		(in_bom yes)
-		(on_board yes)
-		(dnp no)
-		(fields_autoplaced yes)
-		(property "Reference" "D2"
-			(at 195.58 41.8464 90)
-			(effects
-				(font
-					(size 1.27 1.27)
-				)
-				(justify right)
-			)
-		)
-		(property "Value" "LED_Small"
-			(at 195.58 44.3864 90)
-			(effects
-				(font
-					(size 1.27 1.27)
-				)
-				(justify right)
-			)
-		)
-		(property "Footprint" ""
-			(at 193.04 43.18 90)
-			(effects
-				(font
-					(size 1.27 1.27)
-				)
-				(hide yes)
-			)
-		)
-		(property "Datasheet" "~"
-			(at 193.04 43.18 90)
-			(effects
-				(font
-					(size 1.27 1.27)
-				)
-				(hide yes)
-			)
-		)
-		(property "Description" "Light emitting diode, small symbol"
-			(at 193.04 43.18 0)
-			(effects
-				(font
-					(size 1.27 1.27)
-				)
-				(hide yes)
-			)
-		)
-		(pin "1"
-		)
-		(pin "2"
-		)
-		(instances
-			(project "LoRaNode328"
-				(path "/e0ffc31c-24f5-4303-8af9-d0625c9ddd62/c6cbfb80-403d-495c-81c3-fcdf300803b8"
-					(reference "D2")
-					(unit 1)
-				)
-			)
-		)
-	)
-	(symbol
 		(lib_id "Device:C_Small")
 		(at 161.29 147.32 0)
@@
 	(symbol
 		(lib_id "power:GND")
-		(at 193.04 48.26 0)
-		(unit 1)
-		(exclude_from_sim no)
-		(in_bom yes)
-		(on_board yes)
-		(dnp no)
-		(fields_autoplaced yes)
-		(property "Reference" "#PWR01"
-			(at 193.04 54.61 0)
-			(effects
-				(font
-					(size 1.27 1.27)
-				)
-				(hide yes)
-			)
-		)
-		(property "Value" "GND"
-			(at 193.04 53.34 0)
-			(effects
-				(font
-					(size 1.27 1.27)
-				)
-			)
-		)
-		(property "Footprint" ""
-			(at 193.04 48.26 0)
-			(effects
-				(font
-					(size 1.27 1.27)
-				)
-				(hide yes)
-			)
-		)
-		(property "Datasheet" ""
-			(at 193.04 48.26 0)
-			(effects
-				(font
-					(size 1.27 1.27)
-				)
-				(hide yes)
-			)
-		)
-		(property "Description" "Power symbol creates a global label with name \"GND\" , ground"
-			(at 193.04 48.26 0)
-			(effects
-				(font
-					(size 1.27 1.27)
-				)
-				(hide yes)
-			)
-		)
-		(pin "1"
-		)
-		(instances
-			(project "LoRaNode328"
-				(path "/e0ffc31c-24f5-4303-8af9-d0625c9ddd62/c6cbfb80-403d-495c-81c3-fcdf300803b8"
-					(reference "#PWR01")
-					(unit 1)
-				)
-			)
-		)
-	)
-	(symbol
-		(lib_id "power:GND")
 		(at 142.24 119.38 0)
 		(unit 1)
@@
 					(unit 1)
 				)
-			)
-		)
-	)
-	(symbol
-		(lib_id "Device:R_Small")
-		(at 193.04 35.56 0)
-		(unit 1)
-		(exclude_from_sim no)
-		(in_bom yes)
-		(on_board yes)
-		(dnp no)
-		(fields_autoplaced yes)
-		(property "Reference" "R4"
-			(at 195.58 34.2899 0)
-			(effects
-				(font
-					(size 1.27 1.27)
-				)
-				(justify left)
-			)
-		)
-		(property "Value" "4K7"
-			(at 195.58 36.8299 0)
-			(effects
-				(font
-					(size 1.27 1.27)
-				)
-				(justify left)
-			)
-		)
-		(property "Footprint" ""
-			(at 193.04 35.56 0)
-			(effects
-				(font
-					(size 1.27 1.27)
-				)
-				(hide yes)
-			)
-		)
-		(property "Datasheet" "~"
-			(at 193.04 35.56 0)
-			(effects
-				(font
-					(size 1.27 1.27)
-				)
-				(hide yes)
-			)
-		)
-		(property "Description" "Resistor, small symbol"
-			(at 193.04 35.56 0)
-			(effects
-				(font
-					(size 1.27 1.27)
-				)
-				(hide yes)
-			)
-		)
-		(pin "1"
-		)
-		(pin "2"
-		)
-		(instances
-			(project "LoRaNode328"
-				(path "/e0ffc31c-24f5-4303-8af9-d0625c9ddd62/c6cbfb80-403d-495c-81c3-fcdf300803b8"
-					(reference "R4")
-					(unit 1)
-				)
